Commit message: remove dependency on ur_e_description

File: model/ur3e.urdf (robot description, URDF)
Before this commit: robot ur3e, 11 links, 10 joints
Links:
- removed link tool0
- link base_link: geometry collision mesh filename=package://cito/model/mesh/ur3e/collision/base.stl; visual mesh filename=package://cito/model/mesh/ur3e/visual/base.dae
- link forearm_link: geometry collision mesh filename=package://cito/model/mesh/ur3e/collision/forearm.stl; visual mesh filename=package://cito/model/mesh/ur3e/visual/forearm.dae
- link shoulder_link: geometry collision mesh filename=package://cito/model/mesh/ur3e/collision/shoulder.stl; visual mesh filename=package://cito/model/mesh/ur3e/visual/shoulder.dae
- link upper_arm_link: geometry collision mesh filename=package://cito/model/mesh/ur3e/collision/upperarm.stl; visual mesh filename=package://cito/model/mesh/ur3e/visual/upperarm.dae
- link wrist_1_link: geometry collision mesh filename=package://cito/model/mesh/ur3e/collision/wrist1.stl; visual mesh filename=package://cito/model/mesh/ur3e/visual/wrist1.dae
- link wrist_2_link: geometry collision mesh filename=package://cito/model/mesh/ur3e/collision/wrist2.stl; visual mesh filename=package://cito/model/mesh/ur3e/visual/wrist2.dae
- link wrist_3_link: geometry collision mesh filename=package://cito/model/mesh/ur3e/collision/wrist3.stl; visual mesh filename=package://cito/model/mesh/ur3e/visual/wrist3.dae
Joints:
- removed joint wrist_3_link-tool0_fixed_joint
